Commit message: Imported upstream version '2.3.2' of 'upstream'

File: husarion_ugv_description/urdf/common/gazebo.urdf.xacro (robot description, xacro)
@@ -34,4 +34,5 @@
         <ros>
           <namespace>${namespace}</namespace>
+          <remapping>/diagnostics:=diagnostics</remapping>
           <remapping>drive_controller/cmd_vel:=cmd_vel</remapping>
           <remapping>drive_controller/odom:=odometry/wheels</remapping>
@@ -40,4 +41,5 @@
           <remapping>imu_broadcaster/transition_event:=imu_broadcaster/_transition_event</remapping>
           <remapping>joint_state_broadcaster/transition_event:=joint_state_broadcaster/_transition_event</remapping>
+          <remapping>twist_mux_controller/transition_event:=twist_mux_controller/_transition_event</remapping>
         </ros>
       </plugin>
@@ -132,3 +134,18 @@
     </gazebo>
   </xacro:macro>
+  <xacro:macro name="odometry_publisher" params="namespace:=''">
+    <xacro:property name="ns" value='${namespace + "/" if namespace else ""}' />
+    <gazebo>
+      <plugin
+        filename="gz-sim-odometry-publisher-system"
+        name="gz::sim::systems::OdometryPublisher">
+        <odom_frame>world</odom_frame>
+        <robot_base_frame>${ns}base_link</robot_base_frame>
+        <odom_topic>${ns}odometry/ground_truth</odom_topic>
+        <odom_covariance_topic>${ns}odometry/ground_truth_covariance</odom_covariance_topic>
+        <tf_topic>tf_gt</tf_topic>
+        <odom_publish_frequency>50.0</odom_publish_frequency>
+      </plugin>
+    </gazebo>
+  </xacro:macro>
 </robot>

File: husarion_ugv_description/urdf/common/wheel.urdf.xacro (robot description, xacro)
@@ -72,5 +72,5 @@
     <xacro:if value="${use_sim}">
       <xacro:if value="${config['mecanum']}">
-        <gazebo reference="${prefix}_wheel_link" xmlns:ignition="http://ignitionrobotics.org/schema">
+        <gazebo reference="${prefix}_wheel_link" xmlns:gz="http://gazebosim.org/schema">
           <collision>
             <surface>
@@ -79,5 +79,5 @@
                   <mu>1.0</mu>
                   <mu2>0.0</mu2>
-                  <fdir1 ignition:expressed_in="base_link">${fdir}</fdir1>
+                  <fdir1 gz:expressed_in="base_link">${fdir}</fdir1>
                 </ode>
               </friction>

File: husarion_ugv_description/urdf/lynx/lynx_macro.urdf.xacro (robot description, xacro)
@@ -9,5 +9,6 @@
             imu_xyz:='0.052 0.073 -0.006'
             imu_rpy:='0.0 0.0 -1.57'
-            namespace:=''">
+            namespace:=''
+            use_madgwick_filter:=false">
     <xacro:if value="${use_sim}">
       <xacro:property name="imu_xyz" value="0.052 0.073 -0.006" />
@@ -129,4 +130,5 @@
           <param name="data_interval_ms">8</param>
           <param name="callback_delta_epsilon_ms">1</param>
+          <param name="use_madgwick_filter">${use_madgwick_filter}</param>
           <!-- Madgwick Filter Params -->
           <param name="gain">0.00304</param>
@@ -163,4 +165,5 @@
       <!-- <xacro:gazebo.light reference_frame="lights_channel_1_link" name="lights_channel_1" topic="lights/channel_1_frame" namespace="${namespace}" /> -->
       <!-- <xacro:gazebo.light reference_frame="lights_channel_2_link" name="lights_channel_2" topic="lights/channel_2_frame" namespace="${namespace}" /> -->
+      <xacro:gazebo.odometry_publisher namespace="${namespace}" />
     </xacro:if>
   </xacro:macro>

File: husarion_ugv_description/urdf/panther/panther_macro.urdf.xacro (robot description, xacro)
@@ -9,5 +9,6 @@
             imu_xyz:='0.169 0.025 0.092'
             imu_rpy:='0.0 0.0 -1.57'
-            namespace:=''">
+            namespace:=''
+            use_madgwick_filter:=false">
     <xacro:if value="${use_sim}">
       <xacro:property name="imu_xyz" value="-0.195 0.010 0.085" />
@@ -130,4 +131,5 @@
           <param name="data_interval_ms">8</param>
           <param name="callback_delta_epsilon_ms">1</param>
+          <param name="use_madgwick_filter">${use_madgwick_filter}</param>
           <!-- Madgwick Filter Params -->
           <param name="gain">0.00304</param>
@@ -163,4 +165,5 @@
       <xacro:gazebo.light reference_frame="lights_channel_1_link" name="lights_channel_1" topic="lights/channel_1_frame" namespace="${namespace}" />
       <xacro:gazebo.light reference_frame="lights_channel_2_link" name="lights_channel_2" topic="lights/channel_2_frame" namespace="${namespace}" />
+      <xacro:gazebo.odometry_publisher namespace="${namespace}" />
     </xacro:if>
   </xacro:macro>
